File: ROSNin_PCB/ROSNin_PCB.kicad_sch (KiCad schematic)
At the start: 0 parts

Commit message: feat: add Tang Nano 20K footprint and symbol
Parts:
- added U1: Tang_Nano_20K, Custom:TangNano_20K, symbol Custom:Tang_Nano_20K
Changed lines of the file:
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@@
 	(generator_version "9.0")
 	(paper "A4")
+	(symbol
+		(lib_id "Custom:Tang_Nano_20K")
+		(at 139.7 88.9 0)
+		(unit 1)
+		(exclude_from_sim no)
+		(in_bom yes)
+		(on_board yes)
+		(dnp no)
+		(fields_autoplaced yes)
+		(property "Reference" "U1"
+			(at 108.966 127 0)
+			(effects
+				(font
+					(size 1.27 1.27)
+				)
+				(hide yes)
+			)
+		)
+		(property "Value" "Tang_Nano_20K"
+			(at 139.446 139.954 0)
+			(do_not_autoplace yes)
+			(effects
+				(font
+					(size 1.27 1.27)
+				)
+				(hide yes)
+			)
+		)
+		(property "Footprint" "Custom:TangNano_20K"
+			(at 139.7 87.63 0)
+			(effects
+				(font
+					(size 1.27 1.27)
+				)
+				(hide yes)
+			)
+		)
+		(property "Datasheet" "~"
+			(at 120.65 142.24 0)
+			(effects
+				(font
+					(size 1.27 1.27)
+				)
+				(hide yes)
+			)
+		)
+		(property "Description" "Tang Nano 20K"
+			(at 139.192 96.774 90)
+			(effects
+				(font
+					(size 1.27 1.27)
+				)
+				(hide yes)
+			)
+		)
+		(pin "24"
+		)
+		(pin "10"
+		)
+		(pin "32"
+		)
+		(pin "25"
+		)
+		(pin "29"
+		)
+		(pin "33"
+		)
+		(pin "36"
+		)
+		(pin "23"
+		)
+		(pin "35"
+		)
+		(pin "39"
+		)
+		(pin "38"
+		)
+		(pin "1"
+		)
+		(pin "22"
+		)
+		(pin "34"
+		)
+		(pin "3"
+		)
+		(pin "2"
+		)
+		(pin "20"
+		)
+		(pin "12"
+		)
+		(pin "11"
+		)
+		(pin "31"
+		)
+		(pin "4"
+		)
+		(pin "16"
+		)
+		(pin "13"
+		)
+		(pin "40"
+		)
+		(pin "17"
+		)
+		(pin "14"
+		)
+		(pin "27"
+		)
+		(pin "30"
+		)
+		(pin "37"
+		)
+		(pin "18"
+		)
+		(pin "15"
+		)
+		(pin "8"
+		)
+		(pin "28"
+		)
+		(pin "26"
+		)
+		(pin "7"
+		)
+		(pin "19"
+		)
+		(pin "21"
+		)
+		(pin "6"
+		)
+		(pin "5"
+		)
+		(pin "9"
+		)
+		(instances
+			(project "ROSNin_PCB"
+				(path "/4cf227a6-5ff8-4187-adff-9ef30171355a"
+					(reference "U1")
+					(unit 1)
+				)
+			)
+		)
+	)
 	(sheet_instances
 		(path "/"

Commit message: feat: add Tang Nano 20K library for the project
Parts:
- removed U1: Tang_Nano_20K, Custom:TangNano_20K, symbol Custom:Tang_Nano_20K
- added U1: Tang_Nano_20K, Custom:TangNano_20K, symbol TangNano_20K:Tang_Nano_20K
Changed lines of the file:
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@@
 	(paper "A4")
 	(symbol
-		(lib_id "Custom:Tang_Nano_20K")
-		(at 139.7 88.9 0)
+		(lib_id "TangNano_20K:Tang_Nano_20K")
+		(at 149.86 83.82 0)
 		(unit 1)
 		(exclude_from_sim no)
@@
 		(fields_autoplaced yes)
 		(property "Reference" "U1"
-			(at 108.966 127 0)
+			(at 119.126 121.92 0)
 			(effects
 				(font
@@
 		)
 		(property "Value" "Tang_Nano_20K"
-			(at 139.446 139.954 0)
+			(at 149.606 134.874 0)
 			(do_not_autoplace yes)
 			(effects
@@
 		)
 		(property "Footprint" "Custom:TangNano_20K"
-			(at 139.7 87.63 0)
+			(at 149.86 82.55 0)
 			(effects
 				(font
@@
 		)
 		(property "Datasheet" "~"
-			(at 120.65 142.24 0)
+			(at 130.81 137.16 0)
 			(effects
 				(font
@@
 		)
 		(property "Description" "Tang Nano 20K"
-			(at 139.192 96.774 90)
+			(at 149.352 91.694 90)
 			(effects
 				(font
@@
 			)
 		)
-		(pin "24"
+		(pin "38"
 		)
-		(pin "10"
+		(pin "33"
 		)
-		(pin "32"
+		(pin "34"
+		)
+		(pin "20"
 		)
 		(pin "25"
 		)
+		(pin "36"
+		)
+		(pin "4"
+		)
+		(pin "7"
+		)
 		(pin "29"
 		)
-		(pin "33"
+		(pin "16"
 		)
-		(pin "36"
+		(pin "37"
 		)
-		(pin "23"
+		(pin "8"
+		)
+		(pin "40"
+		)
+		(pin "31"
+		)
+		(pin "19"
 		)
 		(pin "35"
 		)
-		(pin "39"
-		)
-		(pin "38"
-		)
-		(pin "1"
-		)
-		(pin "22"
-		)
-		(pin "34"
-		)
-		(pin "3"
-		)
-		(pin "2"
-		)
-		(pin "20"
+		(pin "17"
 		)
 		(pin "12"
@@
 		(pin "11"
 		)
-		(pin "31"
+		(pin "30"
 		)
-		(pin "4"
-		)
-		(pin "16"
+		(pin "14"
 		)
 		(pin "13"
 		)
-		(pin "40"
+		(pin "39"
 		)
-		(pin "17"
+		(pin "10"
 		)
-		(pin "14"
-		)
-		(pin "27"
-		)
-		(pin "30"
-		)
-		(pin "37"
+		(pin "15"
 		)
 		(pin "18"
 		)
-		(pin "15"
+		(pin "9"
 		)
-		(pin "8"
+		(pin "32"
+		)
+		(pin "26"
+		)
+		(pin "22"
+		)
+		(pin "23"
 		)
 		(pin "28"
 		)
-		(pin "26"
+		(pin "3"
 		)
-		(pin "7"
-		)
-		(pin "19"
+		(pin "27"
 		)
 		(pin "21"
@@
 		(pin "5"
 		)
-		(pin "9"
+		(pin "2"
+		)
+		(pin "1"
+		)
+		(pin "24"
 		)
 		(instances
